File: test/files/properties.kicad_pcb (KiCad board)
At the start: 4 copper layers, 0 parts

Commit message: Add text.shown_text with variable expanasion and all that jazz
Parts:
- added FID1: Fiducial_1mm_Mask2mm, Fiducial:Fiducial_1mm_Mask2mm, F.Cu at (0.00, 0.00)
Other:
- board text added: "hello ${var1}"
Changed lines of the file:
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@@
   (property "var2" "var 2 value")
   (net 0 "")
+  (footprint "Fiducial:Fiducial_1mm_Mask2mm" (layer "F.Cu")
+    (at 0 0)
+    (descr "Circular Fiducial, 1mm bare copper, 2mm soldermask opening (Level A)")
+    (tags "fiducial")
+    (property "extra" "An extra property")
+    (attr smd)
+    (fp_text reference "FID1" (at 0 -2) (layer "F.SilkS")
+      (effects (font (size 1 1) (thickness 0.15)))
+    )
+    (fp_text value "Fiducial_1mm_Mask2mm" (at 0 2) (layer "F.Fab")
+      (effects (font (size 1 1) (thickness 0.15)))
+    )
+    (fp_text user "${LAYER} ${extra}" (at 0 4 unlocked) (layer "F.SilkS")
+      (effects (font (size 1 1) (thickness 0.15)))
+    )
+    (fp_text user "${REFERENCE}" (at 0 0) (layer "F.Fab")
+      (effects (font (size 0.4 0.4) (thickness 0.06)))
+    )
+    (fp_circle (center 0 0) (end 1.25 0) (layer "F.CrtYd") (width 0.05) (fill none))
+    (fp_circle (center 0 0) (end 1 0) (layer "F.Fab") (width 0.1) (fill none))
+    (pad "" smd circle (at 0 0) (size 1 1) (layers "F.Cu" "F.Mask")
+      (solder_mask_margin 0.5) (clearance 0.5))
+  )
+  (gr_text "hello ${var1}" (at 0 0) (layer "F.SilkS")
+    (effects (font (size 1.5 1.5) (thickness 0.3)))
+  )
 )
