File: third_party/newstroke/font.sch (KiCad schematic (older format))
At the start: 567 parts

Commit message: Update newstroke with CJK symbols added by KiCAD
Parts:
- removed U?: E_SMALL, symbol E_SMALL
- removed U?: OMEGA_SMALL, symbol OMEGA_SMALL
- U?: symbol DIGIT_0 -> font:DIGIT_0
- U?: symbol DIGIT_1 -> font:DIGIT_1
- U?: symbol DIGIT_2 -> font:DIGIT_2
- U?: symbol DIGIT_3 -> font:DIGIT_3
- U?: symbol DIGIT_4 -> font:DIGIT_4
- U?: symbol DIGIT_5 -> font:DIGIT_5
- U?: symbol DIGIT_6 -> font:DIGIT_6
- U?: symbol DIGIT_7 -> font:DIGIT_7
- U?: symbol DIGIT_8 -> font:DIGIT_8
- U?: symbol DIGIT_9 -> font:DIGIT_9
- U?: symbol QUESTION -> font:QUESTION
- U? (x2): symbol A_CAP -> font:A_CAP
- U?: symbol B_CAP -> font:B_CAP
- U?: symbol C_CAP -> font:C_CAP
- U?: symbol D_CAP -> font:D_CAP
- U?: symbol E_CAP -> font:E_CAP
- U?: symbol F_CAP -> font:F_CAP
- U?: symbol G_CAP -> font:G_CAP
- U?: symbol H_CAP -> font:H_CAP
- U?: symbol I_CAP -> font:I_CAP
- U?: symbol J_CAP -> font:J_CAP
- U?: symbol K_CAP -> font:K_CAP
- U?: symbol L_CAP -> font:L_CAP
- U?: symbol M_CAP -> font:M_CAP
- U?: symbol N_CAP -> font:N_CAP
- U?: symbol O_CAP -> font:O_CAP
- U?: symbol P_CAP -> font:P_CAP
- U?: symbol Q_CAP -> font:Q_CAP
- U?: symbol R_CAP -> font:R_CAP
- U?: symbol S_CAP -> font:S_CAP
- U? (x3): symbol T_CAP -> font:T_CAP
- U?: symbol U_CAP -> font:U_CAP
- U?: symbol V_CAP -> font:V_CAP
- U?: symbol W_CAP -> font:W_CAP
- U?: symbol X_CAP -> font:X_CAP
- U?: symbol Y_CAP -> font:Y_CAP
- U?: symbol Z_CAP -> font:Z_CAP
- U?: symbol SPACE -> symbol:SPACE
- U?: symbol COMMA -> font:COMMA
- U?: symbol FULL_STOP -> font:FULL_STOP
- U?: symbol SEMICOLON -> font:SEMICOLON
- U?: symbol COLON -> font:COLON
- U?: symbol APOSTROPHE -> font:APOSTROPHE
- U?: symbol EXCLAM -> font:EXCLAM
- U?: symbol QUOTE -> font:QUOTE
- U?: symbol SLASH -> font:SLASH
- U?: symbol PAREN -> font:PAREN
- U?: symbol BACKSLASH -> font:BACKSLASH
- U?: symbol BRACE -> font:BRACE
- U?: symbol BRACKET -> font:BRACKET
- U?: symbol AMPERSAND -> font:AMPERSAND
- U?: symbol AT -> font:AT
- U? (x9): symbol A_SMALL -> font:A_SMALL
- U?: symbol B_SMALL -> font:B_SMALL
- U? (x4): symbol C_SMALL -> font:C_SMALL
- U?: symbol D_SMALL -> font:D_SMALL
- U? (x5): symbol E_SMALL -> font:E_SMALL
- U?: symbol F_SMALL -> font:F_SMALL
- U? (x2): symbol G_SMALL -> font:G_SMALL
- U?: symbol H_SMALL -> font:H_SMALL
- U?: symbol I_SMALL -> font:I_SMALL
- U?: symbol J_SMALL -> font:J_SMALL
- U?: symbol K_SMALL -> font:K_SMALL
- U? (x2): symbol L_SMALL -> font:L_SMALL
- U?: symbol M_SMALL -> font:M_SMALL
- U? (x2): symbol N_SMALL -> font:N_SMALL
- U? (x5): symbol O_SMALL -> font:O_SMALL
- U?: symbol P_SMALL -> font:P_SMALL
- U?: symbol Q_SMALL -> font:Q_SMALL
- U? (x2): symbol R_SMALL -> font:R_SMALL
- U? (x2): symbol S_SMALL -> font:S_SMALL
- U? (x3): symbol T_SMALL -> font:T_SMALL
- U?: symbol U_SMALL -> font:U_SMALL
- U? (x2): symbol V_SMALL -> font:V_SMALL
- U?: symbol W_SMALL -> font:W_SMALL
- U?: symbol X_SMALL -> font:X_SMALL
- U?: symbol Y_SMALL -> font:Y_SMALL
- U?: symbol Z_SMALL -> font:Z_SMALL
- U?: symbol GRAVE -> font:GRAVE
- U?: symbol ACUTE -> font:ACUTE
- U?: symbol RING -> font:RING
- U?: symbol CIRCUMFLEX -> font:CIRCUMFLEX
- U?: symbol TILDE -> font:TILDE
- U?: symbol DIAERESIS -> font:DIAERESIS
- U?: symbol AE_CAP -> font:AE_CAP
- U?: symbol AE_SMALL -> font:AE_SMALL
- U?: symbol CEDILLA -> font:CEDILLA
- U?: symbol ESZETT -> font:ESZETT
- U?: symbol ETH_SMALL -> font:ETH_SMALL
- U?: symbol THORN_CAP -> font:THORN_CAP
- U?: symbol THORN_SMALL -> font:THORN_SMALL
- U?: symbol POUND -> font:POUND
- U?: symbol YEN -> font:YEN
- U?: symbol GUILLEMET_DBL -> font:GUILLEMET_DBL
- U?: symbol MACRON -> font:MACRON
- U?: symbol DIGIT_0_SMALL -> font:DIGIT_0_SMALL
- U?: symbol DIGIT_1_SMALL -> font:DIGIT_1_SMALL
- U?: symbol DIGIT_2_SMALL -> font:DIGIT_2_SMALL
- U?: symbol DIGIT_3_SMALL -> font:DIGIT_3_SMALL
- U?: symbol O_TINY -> font:O_TINY
- U?: symbol A_TINY -> font:A_TINY
- U?: symbol SECTION -> font:SECTION
- U?: symbol MU_SMALL -> font:MU_SMALL
- U?: symbol PI_SMALL -> font:PI_SMALL
- U?: symbol O_CAP_STROKE -> font:O_CAP_STROKE
- U?: symbol O_SMALL_STROKE -> font:O_SMALL_STROKE
- U?: symbol OGONEK -> font:OGONEK
- U?: symbol CARON -> font:CARON
- U?: symbol BREVE -> font:BREVE
- U?: symbol L_SMALL_MIDDOT -> font:L_SMALL_MIDDOT
- U?: symbol H_CAP_STROKE -> font:H_CAP_STROKE
- U?: symbol K_SMALLCAP -> font:K_SMALLCAP
- U?: symbol ENG_CAP -> font:ENG_CAP
- U?: symbol ENG_SMALL -> font:ENG_SMALL
- U?: symbol S_LONG_SMALL -> font:S_LONG_SMALL
- U?: symbol GAMMA_CAP -> font:GAMMA_CAP
- U?: symbol DELTA_CAP -> font:DELTA_CAP
- U?: symbol THETA_CAP -> font:THETA_CAP
- U?: symbol LAMBDA_CAP -> font:LAMBDA_CAP
- U?: symbol XI_CAP -> font:XI_CAP
- U? (x2): symbol PI_CAP -> font:PI_CAP
- U?: symbol SIGMA_CAP -> font:SIGMA_CAP
- U?: symbol PHI_CAP -> font:PHI_CAP
- U?: symbol PSI_CAP -> font:PSI_CAP
- U?: symbol OMEGA_CAP -> font:OMEGA_CAP
- U? (x8): symbol ALPHA_SMALL -> font:ALPHA_SMALL
- U?: symbol BETA_SMALL -> font:BETA_SMALL
- U?: symbol GAMMA_SMALL -> font:GAMMA_SMALL
- U?: symbol DELTA_SMALL -> font:DELTA_SMALL
- U?: symbol EPSILON_SMALL -> font:EPSILON_SMALL
- U?: symbol ZETA_SMALL -> font:ZETA_SMALL
- U?: symbol ETA_SMALL -> font:ETA_SMALL
- U?: symbol IOTA_SMALL -> font:IOTA_SMALL
- U?: symbol THETA_SMALL -> font:THETA_SMALL
- U?: symbol LAMBDA_SMALL -> font:LAMBDA_SMALL
- U?: symbol NU_SMALL -> font:NU_SMALL
- U?: symbol XI_SMALL -> font:XI_SMALL
- U?: symbol RHO_SMALL -> font:RHO_SMALL
- U?: symbol SIGMA_SMALL_FINAL -> font:SIGMA_SMALL_FINAL
- U?: symbol SIGMA_SMALL -> font:SIGMA_SMALL
- U?: symbol TAU_SMALL -> font:TAU_SMALL
- U?: symbol UPSILON_SMALL -> font:UPSILON_SMALL
- U?: symbol PHI_SMALL -> font:PHI_SMALL
- U?: symbol CHI_SMALL -> font:CHI_SMALL
- U?: symbol PSI_SMALL -> font:PSI_SMALL
- U? (x3): symbol OMEGA_SMALL -> font:OMEGA_SMALL
- U?: symbol PHI_SMALL_VAR -> font:PHI_SMALL_VAR
- U?: symbol OMEGA_PI_SMALL -> font:OMEGA_PI_SMALL
- U?: symbol BETA_SMALL_CURLED -> font:BETA_SMALL_CURLED
- U?: symbol THETA_SMALL_SCRIPT -> font:THETA_SMALL_SCRIPT
- U?: symbol RHO_SMALL_TAIL -> font:RHO_SMALL_TAIL
- U?: symbol OE_CAP -> font:OE_CAP
- U?: symbol OE_SMALL -> font:OE_SMALL
- U?: symbol KAPPA_SMALL_SCRIPT -> font:KAPPA_SMALL_SCRIPT
- U?: symbol KAI_CAP -> font:KAI_CAP
- U?: symbol KAI_SMALL -> font:KAI_SMALL
- U?: symbol KOPPA_ARCHAIC_CAP -> font:KOPPA_ARCHAIC_CAP
- U?: symbol KOPPA_ARCHAIC_SMALL -> font:KOPPA_ARCHAIC_SMALL
- U?: symbol DIGAMMA_SMALL -> font:DIGAMMA_SMALL
- U?: symbol STIGMA_CAP -> font:STIGMA_CAP
- U?: symbol STIGMA_SMALL -> font:STIGMA_SMALL
- U?: symbol IE_CAP -> font:IE_CAP
- U?: symbol IE_SMALL -> font:IE_SMALL
- U?: symbol C_SMALL_REV -> font:C_SMALL_REV
- U?: symbol C_CAP_REV -> font:C_CAP_REV
- U?: symbol FITA_CAP -> font:FITA_CAP
- U?: symbol FITA_SMALL -> font:FITA_SMALL
- U? (x2): symbol PI_SMALLCAP -> font:PI_SMALLCAP
- U?: symbol Y_LARGE -> font:Y_LARGE
- U?: symbol HETA_CAP -> font:HETA_CAP
- U?: symbol HETA_SMALL -> font:HETA_SMALL
- U?: symbol IZHE_CAP -> font:IZHE_CAP
- U?: symbol IZHE_SMALL -> font:IZHE_SMALL
- U?: symbol SAMPI_ARCHAIC_CAP -> font:SAMPI_ARCHAIC_CAP
- U?: symbol SAMPI_ARCHAIC_SMALL -> font:SAMPI_ARCHAIC_SMALL
- U?: symbol APOSTROPHE_TURNED_LOW -> font:APOSTROPHE_TURNED_LOW
- U?: symbol IOTA_BELOW -> font:IOTA_BELOW
- U?: symbol UPSILON_CAP_HOOK -> font:UPSILON_CAP_HOOK
- U?: symbol KOPPA_CAP -> font:KOPPA_CAP
- U?: symbol KOPPA_SMALL -> font:KOPPA_SMALL
- U?: symbol SAMPI_CAP -> font:SAMPI_CAP
- U?: symbol SAMPI_SMALL -> font:SAMPI_SMALL
- U?: symbol OMEGA_LARGE -> font:OMEGA_LARGE
- U?: symbol SHEI_CAP -> font:SHEI_CAP
- U?: symbol SHEI_SMALL -> font:SHEI_SMALL
- U?: symbol KHEI_CAP -> font:KHEI_CAP
- U?: symbol KHEI_SMALL -> font:KHEI_SMALL
- U?: symbol BUKI_CAP -> font:BUKI_CAP
- U?: symbol BUKI_SMALL -> font:BUKI_SMALL
- U?: symbol ZHIVETE_CAP -> font:ZHIVETE_CAP
- U?: symbol ZHIVETE_SMALL -> font:ZHIVETE_SMALL
- U?: symbol DOBRO_SMALL -> font:DOBRO_SMALL
- U?: symbol DOBRO_CAP -> font:DOBRO_CAP
- U?: symbol ZEMLYA_CAP -> font:ZEMLYA_CAP
- U?: symbol ZEMLYA_SMALL -> font:ZEMLYA_SMALL
- U? (x2): symbol LYUDI_SMALL -> font:LYUDI_SMALL
- U?: symbol LYUDI_CAP -> font:LYUDI_CAP
- U?: symbol M_SMALLCAP -> font:M_SMALLCAP
- U? (x3): symbol H_SMALLCAP -> font:H_SMALLCAP
- U?: symbol TSY_CAP -> font:TSY_CAP
- U?: symbol TSY_SMALL -> font:TSY_SMALL
- U?: symbol FEI_SMALL -> font:FEI_SMALL
- U?: symbol FEI_CAP -> font:FEI_CAP
- U? (x2): symbol CHERV_CAP -> font:CHERV_CAP
- U?: symbol CHERV_SMALL -> font:CHERV_SMALL
- U? (x2): symbol SHA_SMALL -> font:SHA_SMALL
- U?: symbol SHA_CAP -> font:SHA_CAP
- U?: symbol SOFT_CAP -> font:SOFT_CAP
- U?: symbol HARD_CAP -> font:HARD_CAP
- U?: symbol SOFT_SMALL -> font:SOFT_SMALL
- U?: symbol HARD_SMALL -> font:HARD_SMALL
- U?: symbol YERY_SMALL -> font:YERY_SMALL
- U?: symbol YERY_CAP -> font:YERY_CAP
- U?: symbol YU_CAP -> font:YU_CAP
- U?: symbol YU_SMALL -> font:YU_SMALL
- U?: symbol YA_SMALL -> font:YA_SMALL
- U?: symbol YA_CAP -> font:YA_CAP
- U?: symbol B_SMALLCAP -> font:B_SMALLCAP
- U?: symbol GAMMA_SMALLCAP -> font:GAMMA_SMALLCAP
- U?: symbol T_SMALLCAP -> font:T_SMALLCAP
- U?: symbol DIGIT_4_SMALL -> font:DIGIT_4_SMALL
- U?: symbol DIGIT_5_SMALL -> font:DIGIT_5_SMALL
- U?: symbol DIGIT_6_SMALL -> font:DIGIT_6_SMALL
- U?: symbol DIGIT_7_SMALL -> font:DIGIT_7_SMALL
- U?: symbol DIGIT_8_SMALL -> font:DIGIT_8_SMALL
- U?: symbol DIGIT_9_SMALL -> font:DIGIT_9_SMALL
- U?: symbol FLOOR -> font:FLOOR
- U?: symbol DASH_EM -> font:DASH_EM
- U?: symbol SPACE_EM -> font:SPACE_EM
- U?: symbol DASH_EN -> font:DASH_EN
- U?: symbol SPACE_EN -> font:SPACE_EN
- U?: symbol SPACE_THICK -> font:SPACE_THICK
- U?: symbol SPACE_MID -> font:SPACE_MID
- U?: symbol SPACE_THIN -> font:SPACE_THIN
- U?: symbol SPACE_HAIR -> font:SPACE_HAIR
- U?: symbol SPACE_FIGURE -> font:SPACE_FIGURE
- U?: symbol SPACE_PUNC -> font:SPACE_PUNC
- U?: symbol HYPHEN -> font:HYPHEN
- U?: symbol DASH_FIGURE -> font:DASH_FIGURE
- U?: symbol COMMA_DBL -> font:COMMA_DBL
- U?: symbol QUOTE_RIGHT -> font:QUOTE_RIGHT
- U?: symbol QUOTE_RIGHT_DBL -> font:QUOTE_RIGHT_DBL
- U?: symbol I_TINY -> font:I_TINY
- U?: symbol N_TINY -> font:N_TINY
- U?: symbol E_TINY -> font:E_TINY
- U?: symbol X_TINY -> font:X_TINY
- U?: symbol E_TINY_TURNED -> font:E_TINY_TURNED
- U?: symbol PAREN_SMALL -> font:PAREN_SMALL
- U?: symbol GUILLEMET -> font:GUILLEMET
- U?: symbol HORI_CAP -> font:HORI_CAP
- U?: symbol HORI_SMALL -> font:HORI_SMALL
- U?: symbol GANGIA_CAP -> font:GANGIA_CAP
- U?: symbol GANGIA_SMALL -> font:GANGIA_SMALL
- U?: symbol BUKI_LARGE -> font:BUKI_LARGE
- U?: symbol DEI_CAP -> font:DEI_CAP
- U?: symbol DEI_SMALL -> font:DEI_SMALL
- U?: symbol SAN_CAP -> font:SAN_CAP
- U?: symbol SAN_SMALL -> font:SAN_SMALL
- U?: symbol RHO_SMALL_STROKE -> font:RHO_SMALL_STROKE
- U?: symbol DJE_SMALL -> font:DJE_SMALL
- U?: symbol TSHE_SMALL -> font:TSHE_SMALL
- U?: symbol TSHE_CAP -> font:TSHE_CAP
- U?: symbol LJE_CAP -> font:LJE_CAP
- U?: symbol LJE_SMALL -> font:LJE_SMALL
- U?: symbol NJE_CAP -> font:NJE_CAP
- U?: symbol NJE_SMALL -> font:NJE_SMALL
- U?: symbol DZHE_CAP -> font:DZHE_CAP
- U?: symbol DZHE_SMALL -> font:DZHE_SMALL
- U?: symbol YAT_SMALL -> font:YAT_SMALL
- U?: symbol YAT_CAP -> font:YAT_CAP
- U?: symbol IYE_CAP -> font:IYE_CAP
- U?: symbol IYE_SMALL -> font:IYE_SMALL
- U?: symbol YUS_LITTLE_CAP -> font:YUS_LITTLE_CAP
- U?: symbol IYUS_LITTLE_CAP -> font:IYUS_LITTLE_CAP
- U?: symbol YUS_LITTLE_SMALL -> font:YUS_LITTLE_SMALL
- U?: symbol IYUS_LITTLE_SMALL -> font:IYUS_LITTLE_SMALL
- U?: symbol YUS_BIG_CAP -> font:YUS_BIG_CAP
- U?: symbol IYUS_BIG_CAP -> font:IYUS_BIG_CAP
- U?: symbol YUS_BIG_SMALL -> font:YUS_BIG_SMALL
- U?: symbol IYUS_BIG_SMALL -> font:IYUS_BIG_SMALL
- U?: symbol DESCENDER -> font:DESCENDER
- U?: symbol STROKE_SMALL_H -> font:STROKE_SMALL_H
- U?: symbol STROKE_H -> font:STROKE_H
- U?: symbol SLASH_SMALL_H -> font:SLASH_SMALL_H
- U?: symbol Y_SMALL_STRAIGHT -> font:Y_SMALL_STRAIGHT
- U?: symbol STROKE_V -> font:STROKE_V
- U? (x2): symbol HOOK -> font:HOOK
- U?: symbol TAIL -> font:TAIL
- U?: symbol GAMMA_CAP_HOOK -> font:GAMMA_CAP_HOOK
- U?: symbol GAMMA_SMALLCAP_HOOK -> font:GAMMA_SMALLCAP_HOOK
- U?: symbol E_LARGE -> font:E_LARGE
- U?: symbol H_LARGE -> font:H_LARGE
- U?: symbol TTSE_CAP -> font:TTSE_CAP
- U?: symbol TTSE_SMALL -> font:TTSE_SMALL
- U?: symbol CHE_LARGE -> font:CHE_LARGE
- U?: symbol CHE_SMALL -> font:CHE_SMALL
- U?: symbol K_CAP_BASHKIR -> font:K_CAP_BASHKIR
- U?: symbol K_SMALL_BASHKIR -> font:K_SMALL_BASHKIR
- U?: symbol HGAMMA_CAP -> font:HGAMMA_CAP
- U?: symbol HGAMMA_SMALLCAP -> font:HGAMMA_SMALLCAP
- U?: symbol HA_ABKHAZ_CAP -> font:HA_ABKHAZ_CAP
- U?: symbol HA_ABKHAZ_SMALL -> font:HA_ABKHAZ_SMALL
- U?: symbol GAMMA_CAP_UPTURN -> font:GAMMA_CAP_UPTURN
- U?: symbol GAMMA_SMALLCAP_UPTURN -> font:GAMMA_SMALLCAP_UPTURN
- U?: symbol SEMISOFT_SMALL -> font:SEMISOFT_SMALL
- U?: symbol SLASH_SMALL_V -> font:SLASH_SMALL_V
- U?: symbol KSI_CAP -> font:KSI_CAP
- U?: symbol KSI_SMALL -> font:KSI_SMALL
- U?: symbol OMEGA_ROUND_CAP -> font:OMEGA_ROUND_CAP
- U?: symbol OMEGA_ROUND_SMALL -> font:OMEGA_ROUND_SMALL
- U?: symbol POKRYTIE -> font:POKRYTIE
- U?: symbol T_CAP_ABOVE -> font:T_CAP_ABOVE
- U?: symbol KOPPA_CYR_CAP -> font:KOPPA_CYR_CAP
- U?: symbol KOPPA_CYR_SMALL -> font:KOPPA_CYR_SMALL
- U?: symbol GRAVE_DBL -> font:GRAVE_DBL
- U?: symbol EZH_SMALL -> font:EZH_SMALL
- U?: symbol BREVE_INV -> font:BREVE_INV
- U?: symbol TILDE_MACRON -> font:TILDE_MACRON
- U?: symbol DOT_MACRON -> font:DOT_MACRON
- U?: symbol SLASH_CAP -> font:SLASH_CAP
- U?: symbol SLASH_SMALL -> font:SLASH_SMALL
- U?: symbol YOGH_CAP -> font:YOGH_CAP
- U?: symbol YOGH_SMALL -> font:YOGH_SMALL
- U?: symbol OU_SMALL -> font:OU_SMALL
- U?: symbol OU_CAP -> font:OU_CAP
- U?: symbol DB_SMALL -> font:DB_SMALL
- U?: symbol QP_SMALL -> font:QP_SMALL
- U?: symbol WYNN_SMALL -> font:WYNN_SMALL
- U?: symbol WYNN_CAP -> font:WYNN_CAP
- U?: symbol OI_CAP -> font:OI_CAP
- U?: symbol OI_SMALL -> font:OI_SMALL
- U?: symbol D_SMALL_CURL -> font:D_SMALL_CURL
- U?: symbol L_SMALL_CURL -> font:L_SMALL_CURL
- U?: symbol N_SMALL_CURL -> font:N_SMALL_CURL
- U?: symbol T_SMALL_CURL -> font:T_SMALL_CURL
- U?: symbol S_SMALL_SWASHTAIL -> font:S_SMALL_SWASHTAIL
- U?: symbol Z_SMALL_SWASHTAIL -> font:Z_SMALL_SWASHTAIL
- U?: symbol RING_ACUTE -> font:RING_ACUTE
- U?: symbol EZH_SMALL_TAIL -> font:EZH_SMALL_TAIL
- U?: symbol HORN -> font:HORN
- U?: symbol M_LARGE -> font:M_LARGE
- U?: symbol IOTA_LARGE -> font:IOTA_LARGE
- U?: symbol HV_SMALL -> font:HV_SMALL
- U?: symbol YR_CAP -> font:YR_CAP
- U?: symbol ESH_SMALL_LOOP -> font:ESH_SMALL_LOOP
- U?: symbol B_CAP_HOOK -> font:B_CAP_HOOK
- U?: symbol B_SMALL_TOPBAR -> font:B_SMALL_TOPBAR
- U?: symbol D_CAP_HOOK -> font:D_CAP_HOOK
- U?: symbol EPSILON_LARGE -> font:EPSILON_LARGE
- U?: symbol GAMMA_AFR_CAP -> font:GAMMA_AFR_CAP
- U?: symbol K_CAP_HOOK -> font:K_CAP_HOOK
- U?: symbol P_CAP_HOOK -> font:P_CAP_HOOK
- U?: symbol T_CAP_HOOK -> font:T_CAP_HOOK
- U?: symbol T_SMALL_CARON -> font:T_SMALL_CARON
- U?: symbol T_SMALL_HOOK -> font:T_SMALL_HOOK
- U?: symbol UPSILON_LARGE -> font:UPSILON_LARGE
- U?: symbol Y_CAP_HOOK -> font:Y_CAP_HOOK
- U?: symbol Y_SMALL_HOOK -> font:Y_SMALL_HOOK
- U? (x2): symbol LINE_V_LETTER -> font:LINE_V_LETTER
- U?: symbol LINE_V_LETTER_DBL -> font:LINE_V_LETTER_DBL
- U?: symbol STROKE_SMALL_H_DBL -> font:STROKE_SMALL_H_DBL
- U?: symbol DZ_SMALL -> font:DZ_SMALL
- U?: symbol O_CAP_OGONEK -> font:O_CAP_OGONEK
- U?: symbol O_SMALL_OGONEK -> font:O_SMALL_OGONEK
- U?: symbol U_CAP_STROKE -> font:U_CAP_STROKE
- U?: symbol Q_LARGE_TAIL -> font:Q_LARGE_TAIL
- U?: symbol Q_SMALL_TAIL -> font:Q_SMALL_TAIL
- U?: symbol Y_CAP_STROKE -> font:Y_CAP_STROKE
- U?: symbol Y_SMALL_STROKE -> font:Y_SMALL_STROKE
- U?: symbol HV_CAP -> font:HV_CAP
- U?: symbol THOUSANDS_CYR -> font:THOUSANDS_CYR
- U?: symbol TITLO -> font:TITLO
- U?: symbol PALATALIZATION_CYR -> font:PALATALIZATION_CYR
- U?: symbol HUNDRED_THOUSANDS_CYR -> font:HUNDRED_THOUSANDS_CYR
- U?: symbol MILLIONS_CYR -> font:MILLIONS_CYR
- U?: symbol HV_SMALLCAP -> font:HV_SMALLCAP
- U?: symbol G_SMALLCAP -> font:G_SMALLCAP
- U?: symbol TJE_KOMI_CAP -> font:TJE_KOMI_CAP
- U?: symbol TJE_KOMI_SMALL -> font:TJE_KOMI_SMALL
- U?: symbol YAE_CAP -> font:YAE_CAP
- U?: symbol YAE_SMALL -> font:YAE_SMALL
- U?: symbol LYUDIX_CAP -> font:LYUDIX_CAP
- U?: symbol LYUDIX_SMALL -> font:LYUDIX_SMALL
- U?: symbol PX_CAP -> font:PX_CAP
- U?: symbol PX_SMALL -> font:PX_SMALL
- U?: symbol DJE_KOMI_CAP -> font:DJE_KOMI_CAP
- U?: symbol LJE_KOMI_SMALL -> font:LJE_KOMI_SMALL
- U?: symbol DJE_KOMI_SMALL -> font:DJE_KOMI_SMALL
- U?: symbol LJE_KOMI_CAP -> font:LJE_KOMI_CAP
- U?: symbol ZJE_KOMI_CAP -> font:ZJE_KOMI_CAP
- U?: symbol ZJE_KOMI_SMALL -> font:ZJE_KOMI_SMALL
- U?: symbol DZJE_KOMI_SMALL -> font:DZJE_KOMI_SMALL
- U?: symbol DZJE_KOMI_CAP -> font:DZJE_KOMI_CAP
- U?: symbol B_SMALL_HOOK -> font:B_SMALL_HOOK
- U?: symbol C_SMALL_CURL -> font:C_SMALL_CURL
- U?: symbol D_SMALL_HOOK -> font:D_SMALL_HOOK
- U?: symbol E_SMALL_HOOK -> font:E_SMALL_HOOK
- U?: symbol EPSILON_SMALL_HOOK -> font:EPSILON_SMALL_HOOK
- U?: symbol EPSILON_SMALL_CLOSED -> font:EPSILON_SMALL_CLOSED
- U?: symbol G_SMALL_SCRIPT -> font:G_SMALL_SCRIPT
- U?: symbol GAMMA_AFR_SMALL -> font:GAMMA_AFR_SMALL
- U?: symbol GAMMA_AFR_SMALLCAP -> font:GAMMA_AFR_SMALLCAP
- U?: symbol H_SMALL_HOOK -> font:H_SMALL_HOOK
- U?: symbol I_SMALLCAP -> font:I_SMALLCAP
- U?: symbol L_SMALL_BELT -> font:L_SMALL_BELT
- U?: symbol L_SMALL_RETROHOOK -> font:L_SMALL_RETROHOOK
- U?: symbol LEZH_SMALL -> font:LEZH_SMALL
- U?: symbol LEG -> font:LEG
- U?: symbol N_SMALLCAP -> font:N_SMALLCAP
- U?: symbol OE_SMALLCAP -> font:OE_SMALLCAP
- U?: symbol OMEGA_SMALL_CLOSED -> font:OMEGA_SMALL_CLOSED
- U?: symbol R_SMALL_FISHHOOK -> font:R_SMALL_FISHHOOK
- U?: symbol R_SMALLCAP -> font:R_SMALLCAP
- U?: symbol ESH_SMALL -> font:ESH_SMALL
- U?: symbol ESH_SMALL_CURL -> font:ESH_SMALL_CURL
- U?: symbol ESH_SQUAT_SMALL -> font:ESH_SQUAT_SMALL
- U?: symbol OMEGA_SMALLCAP -> font:OMEGA_SMALLCAP
- U?: symbol Y_SMALLCAP -> font:Y_SMALLCAP
- U?: symbol Z_SMALL_CURL -> font:Z_SMALL_CURL
- U?: symbol U_SMALL_STROKE -> font:U_SMALL_STROKE
- U?: symbol T_SMALL_RETROHOOK -> font:T_SMALL_RETROHOOK
- U?: symbol C_CAP_STRETCHED -> font:C_CAP_STRETCHED
- U?: symbol J_SMALL_CURL -> font:J_SMALL_CURL
- U?: symbol L_SMALLCAP -> font:L_SMALLCAP
- U?: symbol DEZH_SMALL -> font:DEZH_SMALL
- U?: symbol DZ_SMALL_CURL -> font:DZ_SMALL_CURL
- U?: symbol TS_SMALL -> font:TS_SMALL
- U?: symbol TESH_SMALL -> font:TESH_SMALL
- U?: symbol TC_SMALL_CURL -> font:TC_SMALL_CURL
- U?: symbol FENG_SMALL -> font:FENG_SMALL
- U?: symbol LS_SMALL -> font:LS_SMALL
- U?: symbol LZ_SMALL -> font:LZ_SMALL
- U?: symbol W_OVER_W -> font:W_OVER_W
- U?: symbol BIDENTAL_PERCUSSIVE -> font:BIDENTAL_PERCUSSIVE
- U?: symbol H_SMALL_RETROHOOK -> font:H_SMALL_RETROHOOK
- U?: symbol EZH_SMALL_CURL -> font:EZH_SMALL_CURL
- U?: symbol INTERROBANG -> font:INTERROBANG
- U?: symbol BULLET_LEFT -> font:BULLET_LEFT
- U?: symbol TIE -> font:TIE
- U?: symbol ABZUEGLICH -> font:ABZUEGLICH
- U?: symbol BRACKET_QUILL -> font:BRACKET_QUILL
- U?: symbol ET_TIRONIAN -> font:ET_TIRONIAN
- U?: symbol ANGLE_BRACKET -> font:ANGLE_BRACKET
- U?: symbol ECU -> font:ECU
- U?: symbol FRAC_LINE -> font:FRAC_LINE
- U?: symbol SHEQUEL_NEW -> font:SHEQUEL_NEW
- U?: symbol EURO -> font:EURO
- U?: symbol SLASH_SMALL_H_DBL -> font:SLASH_SMALL_H_DBL
- U?: symbol PENNY_GERMAN -> font:PENNY_GERMAN
- U?: symbol MIDDLE_HOOK_SMALL -> font:MIDDLE_HOOK_SMALL
- U?: symbol MIDDLE_HOOK_CAP -> font:MIDDLE_HOOK_CAP
- U?: symbol PSILI -> font:PSILI
- U?: symbol DASIA -> font:DASIA
- U?: symbol PSILI_VARIA -> font:PSILI_VARIA
- U?: symbol DASIA_VARIA -> font:DASIA_VARIA
- U?: symbol PSILI_OXIA -> font:PSILI_OXIA
- U?: symbol DASIA_OXIA -> font:DASIA_OXIA
- U?: symbol Y_SMALL_LOOP -> font:Y_SMALL_LOOP
- U?: symbol V_MIDWELSH_SMALL -> font:V_MIDWELSH_SMALL
- U?: symbol V_MIDWELSH_CAP -> font:V_MIDWELSH_CAP
- U?: symbol LL_CAP -> font:LL_CAP
- U?: symbol LL_SMALL -> font:LL_SMALL
- U?: symbol CIRCUMFLEX_HOOK -> font:CIRCUMFLEX_HOOK
- U?: symbol CIRCUMFLEX_ACUTE -> font:CIRCUMFLEX_ACUTE
- U?: symbol CIRCUMFLEX_GRAVE -> font:CIRCUMFLEX_GRAVE
- U?: symbol BREVE_HOOK -> font:BREVE_HOOK
- U?: symbol RING_HALF -> font:RING_HALF
- U?: symbol ACUTE_DOT -> font:ACUTE_DOT
- U?: symbol ESZETT_CAP -> font:ESZETT_CAP
- U?: symbol A_SMALLCAP -> font:A_SMALLCAP
- U?: symbol AE_SMALLCAP -> font:AE_SMALLCAP
- U?: symbol D_SMALLCAP -> font:D_SMALLCAP
- U?: symbol E_SMALLCAP -> font:E_SMALLCAP
- U?: symbol J_SMALLCAP -> font:J_SMALLCAP
- U?: symbol O_SMALL_SIDE -> font:O_SMALL_SIDE
- U?: symbol O_SMALL_STROKE_SIDE -> font:O_SMALL_STROKE_SIDE
- U?: symbol O_SMALL_HALF -> font:O_SMALL_HALF
- U?: symbol P_SMALLCAP -> font:P_SMALLCAP
- U?: symbol U_SMALLCAP -> font:U_SMALLCAP
- U? (x2): symbol U_SMALL_SIDE -> font:U_SMALL_SIDE
- U?: symbol DIAERESIS_SIDE -> font:DIAERESIS_SIDE
- U?: symbol M_SMALL_SIDE -> font:M_SMALL_SIDE
- U?: symbol LAMBDA_SMALLCAP -> font:LAMBDA_SMALLCAP
- U?: symbol PSI_SMALLCAP -> font:PSI_SMALLCAP
- U?: symbol OU_SMALLCAP -> font:OU_SMALLCAP
- U?: symbol A_TINY_TURNED -> font:A_TINY_TURNED
- U?: symbol ALPHA_TINY -> font:ALPHA_TINY
- U?: symbol B_TINY -> font:B_TINY
- U?: symbol D_TINY -> font:D_TINY
- U?: symbol EPSILON_TINY -> font:EPSILON_TINY
- U?: symbol EPSILON_TINY_TURNED -> font:EPSILON_TINY_TURNED
- U?: symbol G_TINY -> font:G_TINY
- U?: symbol K_TINY -> font:K_TINY
- U?: symbol M_TINY -> font:M_TINY
- U?: symbol ENG_TINY -> font:ENG_TINY
- U?: symbol O_TINY_HALF -> font:O_TINY_HALF
- U?: symbol O_TINY_HALF_TOP -> font:O_TINY_HALF_TOP
- U?: symbol P_TINY -> font:P_TINY
- U?: symbol T_TINY -> font:T_TINY
- U?: symbol U_TINY -> font:U_TINY
- U?: symbol U_TINY_SIDE -> font:U_TINY_SIDE
- U?: symbol M_TINY_TURNED -> font:M_TINY_TURNED
- U?: symbol V_TINY -> font:V_TINY
- U?: symbol BETA_TINY -> font:BETA_TINY
- U?: symbol GAMMA_TINY -> font:GAMMA_TINY
- U?: symbol DELTA_TINY -> font:DELTA_TINY
- U?: symbol PHI_TINY -> font:PHI_TINY
- U?: symbol CHI_TINY -> font:CHI_TINY
- U?: symbol R_TINY -> font:R_TINY
- U?: symbol UE_SMALL -> font:UE_SMALL
- U?: symbol EZH_SMALL_LOOP -> font:EZH_SMALL_LOOP
- U?: symbol C_SMALL_SIDE -> font:C_SMALL_SIDE
- U?: symbol AE_TINY_TURNED -> font:AE_TINY_TURNED
- U?: symbol C_TINY_TURNED -> font:C_TINY_TURNED
- U?: symbol GAMMA_AFR_TINYCAP_TURNED -> font:GAMMA_AFR_TINYCAP_TURNED
- U?: symbol RHO_TINY -> font:RHO_TINY
Connections:
- net at U?.~: now also U?.~ (x83)
- net at U?.~: now also U?.~; no longer U?.~ (x256)
- net at U?.~: now also U?.~ (S); no longer U?.~ (x3)
- net at U?.~ (S): now also U?.~; no longer U?.~ (x2)
- net at U?.~: no longer U?.~ (S) (x3)
- net at U?.~: no longer U?.~ (x128)
- net at U?.~ (TONOS): now also U?.~ (x3)
- net at U?.~: now also U?.~; no longer U?.~ (TONOS) (x4)
- net at U?.~ (TOP2): now also U?.~
- net at U?.~: now also U?.~; no longer U?.~ (TOP2)
- net at U?.~ (TONOS): now also U?.~ (S)
- net at U?.~ (S): now also U?.~; no longer U?.~ (TONOS)
- net at U?.~: now also U?.~ (TONOS); no longer U?.~
- net at U?.~ (TONOS): now also U?.~; no longer U?.~ (x2)
- net at U?.~: now also U?.~ (TONOS); no longer U?.~ (TONOS)
- net at U?.~ (S): now also U?.~ (S); no longer U?.~
- net at U?.~ (S): now also U?.~; no longer U?.~ (S)
- net at U?.~: now also U?.~; no longer U?.~ (S)
- net at U?.~ (X): no longer U?.~ (x4)
- net at U?.~: now also U?.~, U?.~; no longer U?.~ (x4)
- net at U?.~: now also U?.~ (S)
- net at U?.~ (S): no longer U?.~
- net at U?.~: now also U?.~ (SAPOS); no longer U?.~
- net at U?.~ (SAPOS): now also U?.~; no longer U?.~
- net at U?.~: no longer U?.~ (SAPOS)
- net at U?.~: now also U?.~ (X2); no longer U?.~ (x3)
- net at U?.~ (X2): no longer U?.~ (x4)
- net at U?.~: now also U?.~ (X); no longer U?.~
- new net: U?.~, U?.~ (x49)
- new net: U?.~, U?.~ (TONOS)
- new net: U?.~, U?.~ (X) (x4)
- new net: U?.~, U?.~ (X2)
- now unconnected: U?.~, U?.~, U?.~, U?.~, U?.~, U?.~, U?.~, U?.~, U?.~, U?.~, U?.~, U?.~, U?.~, U?.~, U?.~, U?.~, U?.~, U?.~, U?.~, U?.~, U?.~, U?.~, U?.~, U?.~, U?.~, U?.~, U?.~, U?.~ (X), U?.~ (X)
Other:
- moved on the sheet: U?
