File: third_party/newstroke/symbols.sch (KiCad schematic (older format))
At the start: 358 parts

Commit message: Update newstroke with CJK symbols added by KiCAD
Parts:
- U?: symbol HASH -> symbol:HASH
- U?: symbol BROKEN_BAR -> symbol:BROKEN_BAR
- U?: symbol REGISTERED -> symbol:REGISTERED
- U?: symbol COPYRIGHT -> symbol:COPYRIGHT
- U?: symbol NOT -> symbol:NOT
- U?: symbol PLUS_MINUS -> symbol:PLUS_MINUS
- U?: symbol DEGREE -> symbol:DEGREE
- U?: symbol CURRENCY -> symbol:CURRENCY
- U? (x2): symbol DIVIDE -> symbol:DIVIDE
- U?: symbol MULTIPLY -> symbol:MULTIPLY
- U?: symbol PERCENT -> symbol:PERCENT
- U?: symbol ASTERISK -> symbol:ASTERISK
- U?: symbol LOW_LINE -> symbol:LOW_LINE
- U? (x6): symbol EQUAL -> symbol:EQUAL
- U?: symbol LESS -> symbol:LESS
- U?: symbol MINUS -> symbol:MINUS
- U?: symbol PLUS -> symbol:PLUS
- U? (x2): symbol ARROW_E -> symbol:ARROW_E
- U?: symbol ARROW_E_STROKE -> symbol:ARROW_E_STROKE
- U?: symbol ARROW_E_SLASH -> symbol:ARROW_E_SLASH
- U?: symbol ARROW_E_BAR -> symbol:ARROW_E_BAR
- U?: symbol ARROW_DBL_E -> symbol:ARROW_DBL_E
- U?: symbol ARROW_E_HOOK -> symbol:ARROW_E_HOOK
- U?: symbol ARROW_E_LOOP -> symbol:ARROW_E_LOOP
- U?: symbol ARROW_E_TAIL -> symbol:ARROW_E_TAIL
- U?: symbol ARROW_E_WAVE -> symbol:ARROW_E_WAVE
- U?: symbol ARROW_N -> symbol:ARROW_N
- U?: symbol ARROW_WE_STROKE -> symbol:ARROW_WE_STROKE
- U?: symbol ARROW_WE_WAVE -> symbol:ARROW_WE_WAVE
- U?: symbol ARROW_E_DASHED -> symbol:ARROW_E_DASHED
- U?: symbol ARROW_NE -> symbol:ARROW_NE
- U?: symbol HARPOON_UP_E -> symbol:HARPOON_UP_E
- U?: symbol ARROW_E_SQUIGGLE -> symbol:ARROW_E_SQUIGGLE
- U?: symbol ARROW_E_DBL -> symbol:ARROW_E_DBL
- U?: symbol ARROW_E_DBL_SLASH -> symbol:ARROW_E_DBL_SLASH
- U?: symbol ARROW_E_WHITE -> symbol:ARROW_E_WHITE
- U?: symbol ARROW_OPEN_E -> symbol:ARROW_OPEN_E
- U?: symbol ARROW_E_STROKE_DBL -> symbol:ARROW_E_STROKE_DBL
- U?: symbol ARROW_WE_STROKE_DBL -> symbol:ARROW_WE_STROKE_DBL
- U?: symbol ARROW_OPEN_WE -> symbol:ARROW_OPEN_WE
- U?: symbol ARROW_E_WALL_WHITE -> symbol:ARROW_E_WALL_WHITE
- U?: symbol ARROW_WE_DBL -> symbol:ARROW_WE_DBL
- U?: symbol ARROW_E_TPL -> symbol:ARROW_E_TPL
- U?: symbol ARROW_BAR_E -> symbol:ARROW_BAR_E
- U?: symbol ARROW_DBL_N -> symbol:ARROW_DBL_N
- U?: symbol ARROW_N_BAR -> symbol:ARROW_N_BAR
- U?: symbol HARPOON_RIGHT_N -> symbol:HARPOON_RIGHT_N
- U?: symbol ARROW_NS_BAR -> symbol:ARROW_NS_BAR
- U?: symbol ARROW_WE_DBL_SLASH -> symbol:ARROW_WE_DBL_SLASH
- U?: symbol ARROW_N_DBL -> symbol:ARROW_N_DBL
- U?: symbol ARROW_N_STROKE_DBL -> symbol:ARROW_N_STROKE_DBL
- U?: symbol ARROW_N_WHITE -> symbol:ARROW_N_WHITE
- U?: symbol ARROW_N_BAR_WHITE -> symbol:ARROW_N_BAR_WHITE
- U?: symbol ARROW_N_PEDESTAL_WHITE -> symbol:ARROW_N_PEDESTAL_WHITE
- U?: symbol ARROW_DBL_N_WHITE -> symbol:ARROW_DBL_N_WHITE
- U?: symbol ARROW_DBL_N_PEDESTAL_WHITE -> symbol:ARROW_DBL_N_PEDESTAL_WHITE
- U?: symbol ARROW_N_PEDESTAL_WHITE_HBAR -> symbol:ARROW_N_PEDESTAL_WHITE_HBAR
- U?: symbol ARROW_N_PEDESTAL_WHITE_VBAR -> symbol:ARROW_N_PEDESTAL_WHITE_VBAR
- U?: symbol ARROW_NS_WHITE -> symbol:ARROW_NS_WHITE
- U?: symbol ARROW_E_N -> symbol:ARROW_E_N
- U?: symbol ARROW_N_E -> symbol:ARROW_N_E
- U?: symbol ARROW_CLOCKWISE_SEMI -> symbol:ARROW_CLOCKWISE_SEMI
- U?: symbol ARROW_CLOCKWISE_OPEN -> symbol:ARROW_CLOCKWISE_OPEN
- U?: symbol ARROW_NE_TOP_BAR -> symbol:ARROW_NE_TOP_BAR
- U?: symbol ARROW_CORNER_NE -> symbol:ARROW_CORNER_NE
- U?: symbol ARROWS_W_E -> symbol:ARROWS_W_E
- U?: symbol TAB -> symbol:TAB
- U?: symbol ARROWS_E_E -> symbol:ARROWS_E_E
- U?: symbol ARROWS_N_S -> symbol:ARROWS_N_S
- U?: symbol ARROWS_N_N -> symbol:ARROWS_N_N
- U?: symbol ARROWS_E_E_E -> symbol:ARROWS_E_E_E
- U?: symbol HARPOONS_W_E -> symbol:HARPOONS_W_E
- U? (x2): symbol CIRCLE -> symbol:CIRCLE
- U?: symbol CIRCLE_LARGE -> symbol:CIRCLE_LARGE
- U?: symbol CIRCLE_LARGE_SLASH -> symbol:CIRCLE_LARGE_SLASH
- U?: symbol ELEMENT -> symbol:ELEMENT
- U?: symbol ELEMENT_SLASH -> symbol:ELEMENT_SLASH
- U?: symbol ELEMENT_SMALL -> symbol:ELEMENT_SMALL
- U?: symbol PI_CAP_HUGE -> symbol:PI_CAP_HUGE
- U?: symbol SIGMA_CAP_HUGE -> symbol:SIGMA_CAP_HUGE
- U?: symbol ASTERISK_OP -> symbol:ASTERISK_OP
- U?: symbol CIRCLE_SMALL -> symbol:CIRCLE_SMALL
- U?: symbol CIRCLE_SMALL_BLACK -> symbol:CIRCLE_SMALL_BLACK
- U?: symbol ANGLE -> symbol:ANGLE
- U?: symbol ANGLE_RIGHT -> symbol:ANGLE_RIGHT
- U?: symbol ANGLE_MEAS -> symbol:ANGLE_MEAS
- U?: symbol ANGLE_ARC -> symbol:ANGLE_ARC
- U?: symbol LINE_V -> symbol:LINE_V
- U?: symbol LINE_V_SLASH -> symbol:LINE_V_SLASH
- U?: symbol LINE_V_DBL -> symbol:LINE_V_DBL
- U?: symbol LINE_V_DBL_SLASH -> symbol:LINE_V_DBL_SLASH
- U?: symbol OR -> symbol:OR
- U?: symbol UNION -> symbol:UNION
- U?: symbol INTEGRAL -> symbol:INTEGRAL
- U?: symbol INTEGRAL_DBL -> symbol:INTEGRAL_DBL
- U?: symbol INTEGRAL_TPL -> symbol:INTEGRAL_TPL
- U?: symbol INTEGRAL_CONTOUR -> symbol:INTEGRAL_CONTOUR
- U?: symbol WAVE -> symbol:WAVE
- U?: symbol SINE -> symbol:SINE
- U?: symbol PROPORTION -> symbol:PROPORTION
- U? (x2): symbol WAVE_MINUS -> symbol:WAVE_MINUS
- U?: symbol ASYMP -> symbol:ASYMP
- U?: symbol S_LAZY -> symbol:S_LAZY
- U?: symbol WREATH_PRODUCT -> symbol:WREATH_PRODUCT
- U? (x2): symbol WAVE_EQUAL -> symbol:WAVE_EQUAL
- U?: symbol WAVE_NOTEQUAL -> symbol:WAVE_NOTEQUAL
- U?: symbol ASYMP_MINUS -> symbol:ASYMP_MINUS
- U?: symbol WAVE_TPL -> symbol:WAVE_TPL
- U?: symbol SLASH_REL -> symbol:SLASH_REL
- U?: symbol SLASH_OP -> symbol:SLASH_OP
- U?: symbol IDENTICAL -> symbol:IDENTICAL
- U?: symbol STRICTEQV -> symbol:STRICTEQV
- U?: symbol PLUS_SMALL -> symbol:PLUS_SMALL
- U?: symbol MINUS_SMALL -> symbol:MINUS_SMALL
- U?: symbol MULTIPLY_SMALL -> symbol:MULTIPLY_SMALL
- U?: symbol EQUAL_SMALL -> symbol:EQUAL_SMALL
- U?: symbol DOT -> symbol:DOT
- U?: symbol LESS_MINUS -> symbol:LESS_MINUS
- U?: symbol LESS_EQUAL -> symbol:LESS_EQUAL
- U?: symbol LESS_NOTEQUAL -> symbol:LESS_NOTEQUAL
- U?: symbol GREATER_NOTEQUAL -> symbol:GREATER_NOTEQUAL
- U?: symbol ANGLE_RIGHT_ARC -> symbol:ANGLE_RIGHT_ARC
- U?: symbol TRIANGLE -> symbol:TRIANGLE
- U?: symbol TRIANGLE_E -> symbol:TRIANGLE_E
- U?: symbol SQUARE -> symbol:SQUARE
- U?: symbol TRIANGLE_TALL -> symbol:TRIANGLE_TALL
- U?: symbol TRIANGLE_TALL_E -> symbol:TRIANGLE_TALL_E
- U?: symbol RATIO -> symbol:RATIO
- U?: symbol THEREFORE -> symbol:THEREFORE
- U?: symbol SUBSET -> symbol:SUBSET
- U?: symbol SQIMAGE -> symbol:SQIMAGE
- U? (x2): symbol SUBSET_MINUS -> symbol:SUBSET_MINUS
- U?: symbol SQIMAGE_MINUS -> symbol:SQIMAGE_MINUS
- U?: symbol SQCUP -> symbol:SQCUP
- U?: symbol UNION_HUGE -> symbol:UNION_HUGE
- U?: symbol OR_HUGE -> symbol:OR_HUGE
- U?: symbol SLASH_SYM -> symbol:SLASH_SYM
- U?: symbol SQUARE_BLACK -> symbol:SQUARE_BLACK
- U?: symbol SQUARE_SMALL -> symbol:SQUARE_SMALL
- U?: symbol SQUARE_SMALL_BLACK -> symbol:SQUARE_SMALL_BLACK
- U?: symbol RECTANGLE_V_HUGE -> symbol:RECTANGLE_V_HUGE
- U?: symbol EQUAL_SLASH -> symbol:EQUAL_SLASH
- U?: symbol RECTANGLE_V_HUGE_SLASH -> symbol:RECTANGLE_V_HUGE_SLASH
- U?: symbol DIAMOND -> symbol:DIAMOND
- U?: symbol DIAMOND_BLACK -> symbol:DIAMOND_BLACK
- U?: symbol RADICAL -> symbol:RADICAL
- U?: symbol DIGIT_3_SMALL -> font:DIGIT_3_SMALL
- U?: symbol INFINITY -> symbol:INFINITY
- U?: symbol PROPORTIONAL -> symbol:PROPORTIONAL
- U?: symbol SQUARE_FILLV -> symbol:SQUARE_FILLV
- U?: symbol SQUARE_FILLH -> symbol:SQUARE_FILLH
- U?: symbol SQUARE_FILLO -> symbol:SQUARE_FILLO
- U?: symbol SQUARE_FILLB -> symbol:SQUARE_FILLB
- U?: symbol SQUARE_FILLS -> symbol:SQUARE_FILLS
- U?: symbol SQUARE_FILLD -> symbol:SQUARE_FILLD
- U?: symbol SQUARE_ROUNDED -> symbol:SQUARE_ROUNDED
- U?: symbol RECTANGLE -> symbol:RECTANGLE
- U?: symbol RECTANGLE_V -> symbol:RECTANGLE_V
- U?: symbol RECTANGLE_BLACK -> symbol:RECTANGLE_BLACK
- U?: symbol RECTANGLE_V_BLACK -> symbol:RECTANGLE_V_BLACK
- U?: symbol PARALLELOGRAM -> symbol:PARALLELOGRAM
- U?: symbol PARALLELOGRAM_BLACK -> symbol:PARALLELOGRAM_BLACK
- U?: symbol TRIANGLE_BLACK -> symbol:TRIANGLE_BLACK
- U?: symbol TRIANGLE_SMALL -> symbol:TRIANGLE_SMALL
- U?: symbol TRIANGLE_SMALL_BLACK -> symbol:TRIANGLE_SMALL_BLACK
- U?: symbol TRIANGLE_E_BLACK -> symbol:TRIANGLE_E_BLACK
- U?: symbol TRIANGLE_E_SMALL -> symbol:TRIANGLE_E_SMALL
- U?: symbol TRIANGLE_E_SMALL_BLACK -> symbol:TRIANGLE_E_SMALL_BLACK
- U?: symbol TRIANGLE_TALL_BLACK -> symbol:TRIANGLE_TALL_BLACK
- U?: symbol TRIANGLE_TALL_E_BLACK -> symbol:TRIANGLE_TALL_E_BLACK
- U?: symbol DIAMOND_SMALL -> symbol:DIAMOND_SMALL
- U?: symbol DIAMOND_SMALL_BLACK -> symbol:DIAMOND_SMALL_BLACK
- U?: symbol LOZENGE -> symbol:LOZENGE
- U?: symbol CIRCLE_DASHED -> symbol:CIRCLE_DASHED
- U?: symbol CIRCLE_BLACK -> symbol:CIRCLE_BLACK
- U?: symbol CIRCLE_FILLV -> symbol:CIRCLE_FILLV
- U?: symbol STAR_SMALL -> symbol:STAR_SMALL
- U?: symbol STAR -> symbol:STAR
- U?: symbol ARROWHEAD_E -> symbol:ARROWHEAD_E
- U?: symbol ARROWHEAD_N -> symbol:ARROWHEAD_N
- U?: symbol ELECTRIC -> symbol:ELECTRIC
- U?: symbol CROP -> symbol:CROP
- U?: symbol TELEPHONE_RECORDER -> symbol:TELEPHONE_RECORDER
- U?: symbol HASH_SYM -> symbol:HASH_SYM
- U?: symbol WATCH -> symbol:WATCH
- U?: symbol SQUISH_QUAD -> symbol:SQUISH_QUAD
- U?: symbol HELM -> symbol:HELM
- U?: symbol PAUSE -> symbol:PAUSE
- U?: symbol INTERRUPT -> symbol:INTERRUPT
- U?: symbol ESCAPE -> symbol:ESCAPE
- U?: symbol MONOSTABLE -> symbol:MONOSTABLE
- U?: symbol HYSTERESIS -> symbol:HYSTERESIS
- U?: symbol OPEN_H -> symbol:OPEN_H
- U?: symbol DIRECT_CURRENT -> symbol:DIRECT_CURRENT
- U?: symbol PERMILLE -> symbol:PERMILLE
- U?: symbol PERMYRIAD -> symbol:PERMYRIAD
- U?: symbol PRIME -> symbol:PRIME
- U?: symbol PRIME_DBL -> symbol:PRIME_DBL
- U?: symbol PRIME_TPL -> symbol:PRIME_TPL
- U?: symbol EQUIVALENT_GEOM -> symbol:EQUIVALENT_GEOM
- U?: symbol EQUIVALENT -> symbol:EQUIVALENT
- U?: symbol DIFFERENCE -> symbol:DIFFERENCE
- U?: symbol LESS_LESS -> symbol:LESS_LESS
- U?: symbol LESS_TPL -> symbol:LESS_TPL
- U?: symbol LESS_MINUS_GREATER -> symbol:LESS_MINUS_GREATER
- U?: symbol LESS_GREATER -> symbol:LESS_GREATER
- U?: symbol LESS_WAVE -> symbol:LESS_WAVE
- U?: symbol GREATER_WAVE -> symbol:GREATER_WAVE
- U?: symbol PRECEDES -> symbol:PRECEDES
- U?: symbol PRECEDESEQ -> symbol:PRECEDESEQ
- U?: symbol PRECEDES_WAVE -> symbol:PRECEDES_WAVE
- U?: symbol SUCCEEDS_WAVE -> symbol:SUCCEEDS_WAVE
- U?: symbol TACK -> symbol:TACK
- U? (x2): symbol TACK_UP -> symbol:TACK_UP
- U?: symbol TACK_UP_LARGE -> symbol:TACK_UP_LARGE
- U?: symbol FLOOR_CAP -> symbol:FLOOR_CAP
- U?: symbol GROUND -> symbol:GROUND
- U?: symbol SQUARE_FOOT -> symbol:SQUARE_FOOT
- U?: symbol PILLOW -> symbol:PILLOW
- U?: symbol OPTION_KEY -> symbol:OPTION_KEY
- U?: symbol ALTERNATIVE_KEY -> symbol:ALTERNATIVE_KEY
- U?: symbol LINE_V_SYM -> symbol:LINE_V_SYM
- U?: symbol INTEGRAL_DBL_CONTOUR -> symbol:INTEGRAL_DBL_CONTOUR
- U?: symbol INTEGRAL_TPL_CONTOUR -> symbol:INTEGRAL_TPL_CONTOUR
- U?: symbol INTEGRAL_CLOCKWISE -> symbol:INTEGRAL_CLOCKWISE
- U?: symbol INTEGRAL_CONTOUR_CLOCKWISE -> symbol:INTEGRAL_CONTOUR_CLOCKWISE
- U?: symbol INTEGRAL_CONTOUR_COUNTERCLOCKWISE -> symbol:INTEGRAL_CONTOUR_COUNTERCLOCKWISE
- U?: symbol EXCESS -> symbol:EXCESS
- U?: symbol COLON_EQUAL -> symbol:COLON_EQUAL
- U?: symbol IMAGEOF -> symbol:IMAGEOF
- U?: symbol EQUAL_DEF -> symbol:EQUAL_DEF
- U?: symbol DELTA_CAP_ABOVE -> symbol:DELTA_CAP_ABOVE
- U?: symbol QUESTION_ABOVE -> symbol:QUESTION_ABOVE
- U?: symbol M_SMALL_ABOVE -> symbol:M_SMALL_ABOVE
- U?: symbol BETWEEN -> symbol:BETWEEN
- U?: symbol SLASH_SMALL -> font:SLASH_SMALL
- U?: symbol DASH_OP_SMALL -> symbol:DASH_OP_SMALL
- U?: symbol ASSERTION -> symbol:ASSERTION
- U?: symbol MODELS -> symbol:MODELS
- U?: symbol TRUE -> symbol:TRUE
- U?: symbol FORCES -> symbol:FORCES
- U?: symbol BAR_VERT_TPL_STILE_RIGHT -> symbol:BAR_VERT_TPL_STILE_RIGHT
- U?: symbol BAR_VERT_DBL_STILE_RIGHT_DBL -> symbol:BAR_VERT_DBL_STILE_RIGHT_DBL
- U?: symbol PRECEDESREL -> symbol:PRECEDESREL
- U?: symbol TRIANGLE_TALL_E_MINUS -> symbol:TRIANGLE_TALL_E_MINUS
- U?: symbol ORIGINAL -> symbol:ORIGINAL
- U?: symbol MULTIMAP -> symbol:MULTIMAP
- U?: symbol TARGET -> symbol:TARGET
- U?: symbol INTERCALATE -> symbol:INTERCALATE
- U?: symbol OR_MINUS -> symbol:OR_MINUS
- U?: symbol MINUS_OR -> symbol:MINUS_OR
- U?: symbol TRIANGLE_RA -> symbol:TRIANGLE_RA
- U?: symbol BOWTIE -> symbol:BOWTIE
- U?: symbol PRODUCT_NORMAL_FACTOR_SEMIDIRECT -> symbol:PRODUCT_NORMAL_FACTOR_SEMIDIRECT
- U?: symbol PRODUCT_SEMIDIRECT -> symbol:PRODUCT_SEMIDIRECT
- U?: symbol OR_CURLY -> symbol:OR_CURLY
- U?: symbol SUBSET_DBL -> symbol:SUBSET_DBL
- U?: symbol UNION_DBL -> symbol:UNION_DBL
- U?: symbol PITCHFORK -> symbol:PITCHFORK
- U?: symbol SLASH_LINE_H -> symbol:SLASH_LINE_H
- U?: symbol ELLIPSIS_MID -> symbol:ELLIPSIS_MID
- U?: symbol ELLIPSIS_VERT -> symbol:ELLIPSIS_VERT
- U?: symbol ELLIPSIS_DIAG -> symbol:ELLIPSIS_DIAG
- U?: symbol ELEMENT_STROKE -> symbol:ELEMENT_STROKE
- U?: symbol ELEMENT_STROKEBAR -> symbol:ELEMENT_STROKEBAR
- U?: symbol ELEMENT_STROKEBAR_SMALL -> symbol:ELEMENT_STROKEBAR_SMALL
- U?: symbol ELEMENT_MINUS -> symbol:ELEMENT_MINUS
- U?: symbol ELEMENT_MINUS_SMALL -> symbol:ELEMENT_MINUS_SMALL
- U?: symbol ELEMENT_DBLSTROKE -> symbol:ELEMENT_DBLSTROKE
- U?: symbol BAG_MEMBERSHIP -> symbol:BAG_MEMBERSHIP
- U?: symbol SQUARE_LEFTHALF_BLACK -> symbol:SQUARE_LEFTHALF_BLACK
- U?: symbol SECTOR -> symbol:SECTOR
- U?: symbol CIRCLE_BLACKQ -> symbol:CIRCLE_BLACKQ
- U?: symbol CIRCLE_LEFTHALF_BLACK -> symbol:CIRCLE_LEFTHALF_BLACK
- U?: symbol CIRCLE_QUAD -> symbol:CIRCLE_QUAD
- U?: symbol CIRCLE_TOPHALF -> symbol:CIRCLE_TOPHALF
- U?: symbol CIRCLE_TOPHALF_BLACK -> symbol:CIRCLE_TOPHALF_BLACK
- U?: symbol CLEAR_KEY -> symbol:CLEAR_KEY
- U?: symbol ERASE_TO_RIGHT -> symbol:ERASE_TO_RIGHT
- U?: symbol BELL -> symbol:BELL
- U?: symbol NBSP_SYM -> symbol:NBSP_SYM
- U?: symbol SPACE_SYM -> symbol:SPACE_SYM
- U?: symbol TRIANGLE_RA_BLACK -> symbol:TRIANGLE_RA_BLACK
- U?: symbol SMILE -> symbol:SMILE
- U?: symbol LOW_LINE_DBL -> symbol:LOW_LINE_DBL
- U?: symbol DIESIS -> symbol:DIESIS
- U?: symbol DOTS_FOUR_VERT -> symbol:DOTS_FOUR_VERT
- U?: symbol DOTS_4 -> symbol:DOTS_4
- U?: symbol DOTS_3 -> symbol:DOTS_3
- U?: symbol DOTS_5 -> symbol:DOTS_5
- U?: symbol CARET_INSERTION -> symbol:CARET_INSERTION
- U?: symbol HOURGLASS -> symbol:HOURGLASS
- U?: symbol LINE_V_WAVY -> symbol:LINE_V_WAVY
- U?: symbol INTEGRAL_TOP -> symbol:INTEGRAL_TOP
- U?: symbol PAREN_TOP -> symbol:PAREN_TOP
- U?: symbol BRACKET_TOP -> symbol:BRACKET_TOP
- U?: symbol BRACE_TOP -> symbol:BRACE_TOP
- U?: symbol BRACE_MIDDLE -> symbol:BRACE_MIDDLE
- U?: symbol MOUSTACHE -> symbol:MOUSTACHE
- U?: symbol BENZENE -> symbol:BENZENE
- U?: symbol BENZENE_RING -> symbol:BENZENE_RING
- U?: symbol CYLINDRICITY -> symbol:CYLINDRICITY
- U?: symbol SYMMETRY -> symbol:SYMMETRY
- U?: symbol DIMENSION_ORIGIN -> symbol:DIMENSION_ORIGIN
- U?: symbol CIRCLE_MID -> symbol:CIRCLE_MID
- U?: symbol SLOPE -> symbol:SLOPE
- U?: symbol I_BEAM -> symbol:I_BEAM
- U?: symbol KEYBOARD -> symbol:KEYBOARD
- U?: symbol TOTAL_RUNOUT -> symbol:TOTAL_RUNOUT
- U?: symbol ALL_AROUND_PROFILE -> symbol:ALL_AROUND_PROFILE
- U?: symbol COMPOSITION -> symbol:COMPOSITION
- U?: symbol UNDO -> symbol:UNDO
- U?: symbol NEXT_PAGE -> symbol:NEXT_PAGE
- U?: symbol LINE_H -> symbol:LINE_H
- U?: symbol FUSE -> symbol:FUSE
- U?: symbol PAREN_OVER -> symbol:PAREN_OVER
- U?: symbol BRACKET_OVER -> symbol:BRACKET_OVER
- U?: symbol BRACE_OVER -> symbol:BRACE_OVER
- U?: symbol TOR_BRACKET_OVER -> symbol:TOR_BRACKET_OVER
- U?: symbol TRAPEZIUM -> symbol:TRAPEZIUM
- U?: symbol LINE_H_3 -> symbol:LINE_H_3
- U?: symbol LINE_H_1 -> symbol:LINE_H_1
- U?: symbol BREVE_METRICAL -> symbol:BREVE_METRICAL
- U? (x2): symbol BREVE_METRICAL_X2 -> symbol:BREVE_METRICAL_X2
- U?: symbol BREVE_METRICAL_JOINED -> symbol:BREVE_METRICAL_JOINED
- U?: symbol OVERLINE_LONG -> symbol:OVERLINE_LONG
- U?: symbol OVERLINE -> symbol:OVERLINE
- U?: symbol ARROW_E_N_WHITE -> symbol:ARROW_E_N_WHITE
- U?: symbol ENTER_SYM -> symbol:ENTER_SYM
- U?: symbol UNDERLINE_CONT -> symbol:UNDERLINE_CONT
- U?: symbol UNDERLINE_DISCONT -> symbol:UNDERLINE_DISCONT
- U?: symbol EMPHASIS -> symbol:EMPHASIS
- U?: symbol TETRASEME_METRICAL -> symbol:TETRASEME_METRICAL
- U?: symbol PENTASEME_METRICAL -> symbol:PENTASEME_METRICAL
- U?: symbol SIGMA_CAP_TOP -> symbol:SIGMA_CAP_TOP
- U?: symbol HEXAGON_H_CAP -> symbol:HEXAGON_H_CAP
- U?: symbol SCREEN_CLEAR -> symbol:SCREEN_CLEAR
- U?: symbol SCREEN_PRINT -> symbol:SCREEN_PRINT
- U?: symbol ANGLE_RIGHT_ARROW_DOWN_ZIGZAG -> symbol:ANGLE_RIGHT_ARROW_DOWN_ZIGZAG
- U?: symbol TRIANGLE_BLACKHALF -> symbol:TRIANGLE_BLACKHALF
- U?: symbol CIRCLE_INVERSE_HALF -> symbol:CIRCLE_INVERSE_HALF
- U?: symbol CIRCLE_SMALL_BLACK_INVERSE -> symbol:CIRCLE_SMALL_BLACK_INVERSE
- U?: symbol ASTERISM -> symbol:ASTERISM
- U?: symbol LINE_V_SMALL -> symbol:LINE_V_SMALL
- U?: symbol LINE_V_CAP -> symbol:LINE_V_CAP
Connections:
- net at U?.~: now also U?.~ (x33)
- net at U?.~: now also U?.~; no longer U?.~ (x255)
- net at U?.~: no longer U?.~ (x36)
- net at U?.~, U?.~: now also U?.~, U?.~; no longer U?.~, U?.~
- net at U?.~, U?.~: now also U?.~; no longer U?.~, U?.~
- net at U?.~: now also U?.~, U?.~
- new net: U?.~, U?.~ (x15)
- new net: U?.~, U?.~, U?.~, U?.~
- new net: U?.~, U?.~, U?.~
- now unconnected: U?.~, U?.~, U?.~, U?.~, U?.~, U?.~, U?.~
